File: vortex-core.sch (KiCad schematic (older format))
At the start: 146 parts

Commit message: cleanup vortex core switch matrix with net names
Connections:
- net labels added: COL1, COL2, COL3, COL4, COL5, COL6, ROW1, ROW2, ROW3, ROW4, ROW5, ROW6, ROW7, ROW8
- wire segments 447 -> 493
