File: vortex-core.sch (KiCad schematic (older format))
At the start: 146 parts

Commit message: working on vortex core schematics
Parts:
- added C10, C13, C23: 10n, symbol C
- added C11, C12: .1u, symbol C
- added C18: 33u, symbol C
- added C19: C, symbol C
- added C20, C30: 47p, symbol C
- added CN2: Conn_01x05, symbol Conn_01x05
- added CN3: USB_OTG, symbol USB_OTG
- added D120: 0, symbol R
- added R100, R98: 10k, symbol R
- added R121: DNP, symbol R
- added R21, R96: 27, symbol R
- added SEL2: Conn_01x02, symbol Conn_01x02
- added U2: MCP1700-3302E_SOT23, TO_SOT_Packages_SMD:SOT-23, symbol MCP1700-3302E_SOT23
- gave numbers to parts that had none: 5
Connections:
- net labels added: 3.3V, COL7, COL8
- wire segments 493 -> 505
- no-connect marks 0 -> 1
Other:
- note added: "4 Mbit Serial Flash"
- note added: "Debug"
- note added: "SPI1_MISO"
- note added: "SPI1_MOSI"
- note added: "SPI1_SCK"
- note added: "SPI1_SEL"
- note added: "UR0_RX"
- note added: "UR0_TX"
- note added: "UR1_RX"
- note added: "UR1_TX"
- note added: "USR0_RX"
- note added: "USR0_TX"
- note added: "USR1_RX"
- note added: "USR1_TX"

Commit message: Vortex core work
Parts:
- added D118: DNP, symbol D
- added Q77: DNP PNP, TO_SOT_Packages_SMD:SOT-23, symbol BC807
- added R109, R110: DNP, symbol R
Connections:
- wire segments 505 -> 612
- no-connect marks 1 -> 0
Other:
- note added: "wtf was this supposed to do"
- moved on the sheet: U2

Commit message: Add pok3r LED matrix, mostly done
Connections:
- wire segments 612 -> 520

Commit message: schematic library cleanup
Parts:
- C10, C11, C12, C13, C18, C19, C20, C23, C30: symbol C -> chaos-device:C
- CN2: symbol Conn_01x05 -> Connector_Generic:Conn_01x05
- CN3: symbol USB_OTG -> Connector_Specialized:USB_OTG
- D118, D? (x47): symbol D -> chaos-device:D
- D120, R100, R109, R110, R121, R21, R96, R98: symbol R -> chaos-device:R
- D? (x47): symbol LED_RAGB -> chaos-device:LED_RAGB
- Q77: symbol BC807 -> Transistor_BJT:BC807
- S? (x47): symbol MX1A -> mx1a:MX1A
- SEL2: symbol Conn_01x02 -> Connector_Generic:Conn_01x02
- U10: symbol HT32F1654 -> chaos-ic:HT32F1654
- U2: symbol MCP1700-3302E_SOT23 -> Regulator_Linear:MCP1700-3302E_SOT23
- U4: symbol HCT138 -> chaos-ic:HCT138
- U5: symbol GD25Q -> chaos-ic:GD25Q
- U7, U8: symbol MBIA043GP -> chaos-ic:MBIA043GP
Connections:
- wire segments 520 -> 619

Commit message: pok3r_rgb: RGB matrix and LED drivers
Parts:
- added J3, J4: Conn_01x07, symbol Connector_Generic:Conn_01x07
- renumbered SEL2 to SEL1
Connections:
- net +3V3: now also J4.7 (Pin_7)
- net COL5: now also S?.2
- net GND: now also J3.1 (Pin_1)
- net at U10.29 (PD2): now also J3.6 (Pin_6)
- net at U10.32 (PC2): now also J4.4 (Pin_4)
- net at U10.33 (PC3): now also J4.3 (Pin_3)
- net at SEL1.1 (Pin_1), U10.35 (BOOT1/PA9): now also J4.5 (Pin_5)
- net at U10.44 (PB0): now also J3.7 (Pin_7)
- net at U10.49 (PB2): now also J3.2 (Pin_2)
- net at U10.50 (PB3): now also J3.3 (Pin_3)
- net at U10.51 (PB4): now also J3.4 (Pin_4)
- net at U10.52 (PB5): now also J3.5 (Pin_5)
- net at U10.53 (PC7): now also J4.2 (Pin_2)
- net at U10.54 (PC8): now also J4.1 (Pin_1)
- net COL8: no longer names the net of U10.4 (PA3)
- net COL8: no longer S?.2
Changed lines of the file:
@@
 EESchema Schematic File Version 4
-LIBS:vortex-core-cache
 EELAYER 26 0
 EELAYER END
@@
 Debug
 $Comp
-L Connector_Generic:Conn_01x02 SEL2
+L Connector_Generic:Conn_01x02 SEL1
 U 1 1 5A7CC14F
 P 23600 18700
-F 0 "SEL2" H 23600 18800 50  0000 C CNN
+F 0 "SEL1" H 23600 18800 50  0000 C CNN
 F 1 "Conn_01x02" H 23600 18500 50  0001 C CNN
 F 2 "" H 23600 18700 50  0001 C CNN
@@
 COL7
 Text GLabel 2800 11000 3    60   Input ~ 0
-COL8
+COL5
 Text GLabel 18850 17500 0    60   Input ~ 0
 COL7
-Text GLabel 18850 17700 0    60   Input ~ 0
-COL8
 $Comp
 L power:+3.3V #PWR?
@@
 	10900 9100 10900 8850
 Wire Wire Line
-	19550 17700 18850 17700
-Wire Wire Line
 	2800 11000 2800 10000
 Wire Wire Line
@@
 	20550 19950 20550 19550
 Wire Wire Line
-	22450 18700 23400 18700
+	22450 18700 23050 18700
 Wire Wire Line
 	23400 18800 23300 18800
@@
 	22450 18200 24150 18200
 Wire Wire Line
-	24150 18200 24150 17900
+	24150 18200 24150 18000
 Wire Wire Line
-	24150 17900 26100 17900
+	24150 18000 26100 18000
 Wire Wire Line
-	26100 17900 26100 12850
+	26100 18000 26100 12850
 Wire Wire Line
 	22450 18100 24050 18100
 Wire Wire Line
-	24050 18100 24050 17800
+	24050 18100 24050 17900
 Wire Wire Line
-	24050 17800 26200 17800
+	24050 17900 26200 17900
 Wire Wire Line
-	26200 17800 26200 12850
+	26200 17900 26200 12850
 Wire Wire Line
 	24750 16100 24450 16100
@@
 Wire Wire Line
 	7400 10550 9900 10550
+$Comp
+L Connector_Generic:Conn_01x07 J3
+U 1 1 5B2C66BD
+P 17500 13550
+F 0 "J3" H 17420 13117 50  0000 C CNN
+F 1 "Conn_01x07" H 17420 13116 50  0001 C CNN
+F 2 "" H 17500 13550 50  0001 C CNN
+F 3 "~" H 17500 13550 50  0001 C CNN
+	1    17500 13550
+	-1   0    0    1
+$EndComp
+$Comp
+L Connector_Generic:Conn_01x07 J4
+U 1 1 5B2C773D
+P 17500 14900
+F 0 "J4" H 17420 14467 50  0000 C CNN
+F 1 "Conn_01x07" H 17420 14466 50  0001 C CNN
+F 2 "" H 17500 14900 50  0001 C CNN
+F 3 "~" H 17500 14900 50  0001 C CNN
+	1    17500 14900
+	-1   0    0    1
+$EndComp
+$Comp
+L power:+3.3V #PWR?
+U 1 1 5B2CC4EF
+P 17800 14500
+F 0 "#PWR?" H 17800 14350 50  0001 C CNN
+F 1 "+3.3V" H 17815 14673 50  0000 C CNN
+F 2 "" H 17800 14500 50  0001 C CNN
+F 3 "" H 17800 14500 50  0001 C CNN
+	1    17800 14500
+	1    0    0    -1
+$EndComp
+Wire Wire Line
+	17700 14600 17800 14600
+Wire Wire Line
+	17800 14600 17800 14500
+$Comp
+L power:GND #PWR?
+U 1 1 5B32E9D0
+P 17800 13950
+F 0 "#PWR?" H 17800 13700 50  0001 C CNN
+F 1 "GND" H 17805 13777 50  0000 C CNN
+F 2 "" H 17800 13950 50  0001 C CNN
+F 3 "" H 17800 13950 50  0001 C CNN
+	1    17800 13950
+	1    0    0    -1
+$EndComp
+Wire Wire Line
+	17700 13850 17800 13850
+Wire Wire Line
+	17800 13850 17800 13950
+Wire Wire Line
+	17700 13650 21650 13650
+Wire Wire Line
+	21650 13650 21650 16650
+Wire Wire Line
+	17700 13750 21750 13750
+Wire Wire Line
+	21750 13750 21750 16650
+Wire Wire Line
+	17700 13550 21550 13550
+Wire Wire Line
+	21550 13550 21550 16650
+Wire Wire Line
+	17700 13450 21450 13450
+Wire Wire Line
+	21450 13450 21450 16650
+Wire Wire Line
+	17700 13350 25500 13350
+Wire Wire Line
+	25500 13350 25500 20050
+Wire Wire Line
+	25500 20050 21450 20050
+Wire Wire Line
+	21450 20050 21450 19550
+Wire Wire Line
+	17700 13250 25600 13250
+Wire Wire Line
+	25600 13250 25600 17800
+Wire Wire Line
+	25600 17800 22450 17800
+Wire Wire Line
+	21250 16650 21250 15200
+Wire Wire Line
+	21250 15200 17700 15200
+Wire Wire Line
+	17700 15100 21350 15100
+Wire Wire Line
+	21350 15100 21350 16650
+Wire Wire Line
+	17700 15000 25700 15000
+Wire Wire Line
+	25700 15000 25700 19200
+Wire Wire Line
+	25700 19200 22850 19200
+Wire Wire Line
+	22850 19200 22850 18900
+Wire Wire Line
+	22850 18900 22450 18900
+Wire Wire Line
+	17700 14900 25800 14900
+Wire Wire Line
+	25800 14900 25800 20150
+Wire Wire Line
+	25800 20150 21750 20150
+Wire Wire Line
+	21750 20150 21750 19550
+Wire Wire Line
+	17700 14800 25900 14800
+Wire Wire Line
+	25900 14800 25900 19300
+Wire Wire Line
+	25900 19300 23050 19300
+Wire Wire Line
+	23050 19300 23050 18700
+Connection ~ 23050 18700
+Wire Wire Line
+	23050 18700 23400 18700
 $EndSCHEMATC
