File: pok3r-rgb.sch (KiCad schematic (older format))
At the start: 146 parts

Commit message: add poker, vortex tester schematics
Parts:
- removed D?: D110, symbol D
- removed D?: D6, symbol D
- removed D?: D31, symbol D
- removed D?: D23, symbol D
- removed D?: D11, symbol D
- removed D?: D21, symbol D
- removed D?: D111, symbol D
- removed D?: D35, symbol D
- removed D?: D46, symbol D
- removed D?: D112, symbol D
- removed D?: D73, symbol D
- removed D?: D59, symbol D
- removed S? (x12): MX1A, mx1a:MX1A, symbol MX1A
- added D?: D1, symbol D
- added D?: D52_1045, symbol D
- added D?: D9, symbol D
- added D?: D46_1045, symbol D
- added D?: D18, symbol D
- added D?: D12, symbol D
- added D?: D56, symbol D
- added D?: D55, symbol D
- added D?: D54, symbol D
- added D?: D32, symbol D
- added D?: D31, symbol D
- added D?: D30, symbol D
- added D?: D29, symbol D
- added D?: D28, symbol D
- added D?: D27, symbol D
- added D?: D26, symbol D
- added D?: D58, symbol D
- added D?: D57, symbol D
- added D?: D62_105, symbol D
- added D?: D25_1045, symbol D
- added D?: D62, symbol D
- added D?: D61, symbol D
- added D?: D60, symbol D
- added D?: D59, symbol D
- added D?: D53, symbol D
- added D?: D35, symbol D
- added D?: D34, symbol D
- added D?: D33, symbol D
- added S? (x32): MX1A, mx1a:MX1A, symbol MX1A
- D?: value D55 -> D40
- D?: value D32 -> D41
- D?: value D67 -> D39
- D?: value D53 -> D38
- D?: value D66 -> D37
- D?: value D52 -> D36
- D?: value D65 -> D8
- D?: value D51 -> D7
- D?: value D64 -> D6
- D?: value D50 -> D5
- D?: value D63 -> D4
- D?: value D49 -> D3
- D?: value D43 -> D47
- D?: value D41 -> D45
- D?: value D29 -> D44
- D?: value D40 -> D43
- D?: value D28 -> D42
- D?: value D39 -> D16
- D?: value D27 -> D15
- D?: value D38 -> D14
- D?: value D26 -> D13
- D?: value D37 -> D12
- D?: value D25 -> D11
- D?: value D36 -> D10
- D?: value D30 -> D51
- D?: value D16 -> D50
- D?: value D20 -> D49
- D?: value D15 -> D48
- D?: value D19 -> D24
- D?: value D14 -> D23
- D?: value D18 -> D22
- D?: value D13 -> D21
- D?: value D17 -> D20
- D?: value D12 -> D19
- D?: value D62 -> D2
Connections:
- wire segments 493 -> 391
Other:
- moved on the sheet: D?, S?

Commit message: upgrade to kicad 5
Parts:
- removed D?: D40, symbol D
- removed D?: D41, symbol D
- removed D?: D39, symbol D
- removed D?: D38, symbol D
- removed D?: D37, symbol D
- removed D?: D36, symbol D
- removed D?: D8, symbol D
- removed D?: D7, symbol D
- removed D?: D6, symbol D
- removed D?: D5, symbol D
- removed D?: D4, symbol D
- removed D?: D3, symbol D
- removed D?: D47, symbol D
- removed D?: D45, symbol D
- removed D?: D44, symbol D
- removed D?: D43, symbol D
- removed D?: D42, symbol D
- removed D?: D16, symbol D
- removed D?: D15, symbol D
- removed D?: D14, symbol D
- removed D?: D13, symbol D
- removed D? (x2): D12, symbol D
- removed D?: D11, symbol D
- removed D?: D10, symbol D
- removed D?: D51, symbol D
- removed D?: D50, symbol D
- removed D?: D49, symbol D
- removed D?: D48, symbol D
- removed D?: D24, symbol D
- removed D?: D23, symbol D
- removed D?: D22, symbol D
- removed D?: D21, symbol D
- removed D?: D20, symbol D
- removed D?: D19, symbol D
- removed D?: D2, symbol D
- removed D?: D1, symbol D
- removed D?: D52_1045, symbol D
- removed D?: D9, symbol D
- removed D?: D46_1045, symbol D
- removed D?: D18, symbol D
- removed D?: D56, symbol D
- removed D?: D55, symbol D
- removed D?: D54, symbol D
- removed D?: D32, symbol D
- removed D?: D31, symbol D
- removed D?: D30, symbol D
- removed D?: D29, symbol D
- removed D?: D28, symbol D
- removed D?: D27, symbol D
- removed D?: D26, symbol D
- removed D?: D58, symbol D
- removed D?: D57, symbol D
- removed D?: D62_105, symbol D
- removed D?: D25_1045, symbol D
- removed D?: D62, symbol D
- removed D?: D61, symbol D
- removed D?: D60, symbol D
- removed D?: D59, symbol D
- removed D?: D53, symbol D
- removed D?: D35, symbol D
- removed D?: D34, symbol D
- removed D?: D33, symbol D
- removed S? (x67): MX1A, mx1a:MX1A, symbol MX1A
- removed U?: HCT138, MODULE, symbol HCT138
- added C? (x4): C, symbol chaos-device:C
- added CN3: Conn_01x05, symbol Connector_Generic:Conn_01x05
- added CN5: USB_OTG, symbol Connector_Specialized:USB_OTG
- added D1, D16, D17, D24, D242, D244, D246, D248, D25_1045, D26, D32, D33, D34, D35, D36, D37, D38, D39, D40, D41, D42, D45, D46_1045, D47, D48, D51, D52_1045, D53, D54, D56, D57, D58, D59, D60, D61, D62, D62_?, D8, D9, D? (x28): D, symbol chaos-device:D
- added J1: Conn_01x19_Male, symbol Connector_Generic:Conn_01x19
- added J1: Conn_01x19_Female, symbol Connector_Generic:Conn_01x19
- added K25_? (x2), K46_? (x2), K52_? (x2), K63_?, K? (x60): MX1A, mx1a:MX1A, symbol mx1a:MX1A
- added SEL1, SEL2: Conn_01x02, symbol Connector_Generic:Conn_01x02
- added SW?: DIP_SW_QUAD, symbol Switch:SW_DIP_x04
- added U10: MCP1700-3302E_SOT23, TO_SOT_Packages_SMD:SOT-23, symbol pok3r-rescue:MCP1700-3302E_SOT23
- D? (x47): symbol LED_RAGB -> chaos-device:LED_RAGB
- U11, U8: renamed from U?; symbol MBIA043GP -> chaos-ic:MBIA043GP
- U4: renamed from U?; symbol HT32F1654 -> chaos-ic:HT32F1654
- U7: renamed from U?; symbol GD25Q -> chaos-ic:GD25Q
Connections:
- net labels added: 3.3V, COL7, COL8, ROW10, ROW9
- wire segments 391 -> 811
- no-connect marks 0 -> 1
Other:
- note added: "DIP Switches"
- note added: "Debug"
- moved on the sheet: U11, U4, U7, U8

Commit message: schematic library cleanup
Parts:
- U10: symbol pok3r-rescue:MCP1700-3302E_SOT23 -> Regulator_Linear:MCP1700-3302E_SOT23
- gave numbers to parts that had none: 1
Other:
- moved on the sheet: D?
