File: pok3r-rgb.sch (KiCad schematic (older format))
At the start: 197 parts, among them CN3 Conn_01x05, CN5 USB_OTG, J1 Conn_01x19_Female, J1 Conn_01x19_Male, K25_? MX1A, K46_? MX1A, K52_? MX1A, K63_? MX1A, SW1 DIP_SW_QUAD, U10 MCP1700-3302E_SOT23, U11 MBIA043GP, U4 HT32F1654, U7 GD25Q, U8 MBIA043GP

Commit message: pok3r_rgb: RGB matrix and LED drivers
Parts:
- removed D? (x46): LED_RAGB, symbol chaos-device:LED_RAGB
- added C47: C, symbol chaos-device:C
- added D100, D101, D102, D103, D104, D105, D106', D107, D116, D117, D118, D119, D120, D121, D123, D124, D17, D18, D19, D2, D20, D21, D22, D24, D28, D3, D33, D34, D35, D36, D37, D38, D39, D4, D40, D41, D5, D52, D53, D54, D55, D56, D57, D58, D59, D6, D60, D68, D69, D70, D71, D72, D73, D74, D75, D76, D84, D85, D87 (x2), D88, D89, D90, D91, D92: LED_RAGB, symbol chaos-device:LED_RAGB
- added Q1, Q2, Q3, Q4, Q5, Q6, Q7, Q74, Q8: Q_NPN_BCE, symbol Device:Q_NPN_BCE
- added R1, R10, R15, R16, R18, R19, R2, R22, R23, R241, R242, R26, R27, R28, R29, R41, R42 (x2), R6, R68, R7, R70, R71, R9: 1k, symbol Device:R_US
- added R11, R17, R20, R24, R25, R3, R31, R8: 4.7k, symbol Device:R_US
- added R287, R288: 10k, symbol Device:R_US
- added R295, R296, R297, R298, R299, R300, R301, R302, R306: 75, symbol Device:R_US
- added R303, R304, R305, R307, R308, R309, R310, R311, R314, R316, R318, R319, R320, R321, R322, R323, R325, R326: 20, symbol Device:R_US
- added R44, R72: 680, symbol Device:R_US
- added R55, R69: 750, symbol Device:R_US
- CN5: symbol Connector_Specialized:USB_OTG -> pok3r-rgb-rescue:USB_OTG-Connector_Specialized
- gave numbers to parts that had none: 101
- renumbered SEL2 to SEL3, SEL1 to SEL4
Connections:
- net labels added: +5V, GCLK, LED_COL1, LED_COL2, LED_COL3, LED_COL4, LED_COL5, LED_COL6, LED_COL7, LED_COL8, LED_ROW1_B, LED_ROW1_G, LED_ROW1_R, LED_ROW2_B, LED_ROW2_G, LED_ROW2_R, LED_ROW3_B, LED_ROW3_G, LED_ROW3_R, LED_ROW4_B, LED_ROW4_G, LED_ROW4_R, LED_ROW5_B, LED_ROW5_G, LED_ROW5_R, LED_ROW6_B, LED_ROW6_G, LED_ROW6_R, LED_ROW7_B, LED_ROW7_G, LED_ROW7_R, LED_ROW8_B, LED_ROW8_G, LED_ROW8_R, LED_ROW9_B, LED_ROW9_G, LED_ROW9_R, SDI, SDO, VLED
- wire segments 811 -> 1805
- no-connect marks 1 -> 5
Other:
- note added: "CYKB167_D_V03"
- note added: "CYKB167_U_V03"
- moved on the sheet: C38, C39, C40, C41, CN5, D1, D10, D11, D12, D13, D14, D15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
