File: pok3r.sch (KiCad schematic (older format))
At the start: 182 parts

Commit message: pok3r components, need usart tx
Parts:
- removed D? (x47): LED_RAGB, symbol LED_RAGB
- removed U?: HT32F1654, MODULE, symbol HT32F1654
- added D?: SD2, symbol D
- added D?: SD3, symbol D
- added D?: SD4, symbol D
- added D?: SD1, symbol D
- added SEL1, SEL2: CONN_01X02, symbol CONN_01X02
- added SW1: DIP_SW_QUAD, symbol DIP_SW_QUAD
- added U3: HT32F1655, MODULE, symbol HT32F1655
- added Y?: Crystal_GND24, symbol Crystal_GND24
- gave numbers to parts that had none: 1
Connections:
- net labels added: 3.3V
- wire segments 391 -> 432
Other:
- note added: "UR0_RX"
- note added: "UR0_TX"
- note added: "UR1_RX"
- note added: "UR1_TX"
- note added: "USR0_RX"
- note added: "USR0_TX"
- note added: "USR1_RX"
- note added: "USR1_TX"
- moved on the sheet: D?, S?, U?

Commit message: finish pok3r key matrix, connectors
Parts:
- removed U? (x2): MBIA043GP, MODULE, symbol MBIA043GP
- removed U?: HCT138, MODULE, symbol HCT138
- added CN1: USB_OTG, symbol USB_OTG
- added CN2: CONN_01X05, symbol CONN_01X05
- D?: value D12 -> D17
- gave numbers to parts that had none: 62
Connections:
- net labels added: COL7, COL8, ROW9
- wire segments 432 -> 582
Other:
- note added: "4 Mbit Serial Flash"
- note added: "DIP Switches"
- note added: "Debug"
- moved on the sheet: D?, K1, K10, K11, K12, K13, K14, K15, K16, K17, K18, K19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

Commit message: library cleanup, pok3r matric cleanup
Parts:
- D1: renamed from D?; value D1 -> D
- D10: renamed from D?; value D10 -> D
- D11: renamed from D?; value D11 -> D
- D12: renamed from D?; value D12 -> D
- D13: renamed from D?; value D13 -> D
- D14: renamed from D?; value D14 -> D
- D15: renamed from D?; value D15 -> D
- D16: renamed from D?; value D16 -> D
- D17: renamed from D?; value D17 -> D
- D18: renamed from D?; value D18 -> D
- D19: renamed from D?; value D19 -> D
- D2: renamed from D?; value D2 -> D
- D20: renamed from D?; value D20 -> D
- D21: renamed from D?; value D21 -> D
- D22: renamed from D?; value D22 -> D
- D23: renamed from D?; value D23 -> D
- D24: renamed from D?; value D24 -> D
- D25_1045: renamed from D?; value D25_1045 -> D
- D26: renamed from D?; value D26 -> D
- D27: renamed from D?; value D27 -> D
- D28: renamed from D?; value D28 -> D
- D29: renamed from D?; value D29 -> D
- D3: renamed from D?; value D3 -> D
- D30: renamed from D?; value D30 -> D
- D31: renamed from D?; value D31 -> D
- D32: renamed from D?; value D32 -> D
- D33: renamed from D?; value D33 -> D
- D34: renamed from D?; value D34 -> D
- D35: renamed from D?; value D35 -> D
- D36: renamed from D?; value D36 -> D
- D37: renamed from D?; value D37 -> D
- D38: renamed from D?; value D38 -> D
- D39: renamed from D?; value D39 -> D
- D4: renamed from D?; value D4 -> D
- D40: renamed from D?; value D40 -> D
- D41: renamed from D?; value D41 -> D
- D42: renamed from D?; value D42 -> D
- D43: renamed from D?; value D43 -> D
- D44: renamed from D?; value D44 -> D
- D45: renamed from D?; value D45 -> D
- D46_1045: renamed from D?; value D46_1045 -> D
- D47: renamed from D?; value D47 -> D
- D48: renamed from D?; value D48 -> D
- D49: renamed from D?; value D49 -> D
- D5: renamed from D?; value D5 -> D
- D50: renamed from D?; value D50 -> D
- D51: renamed from D?; value D51 -> D
- D52_1045: renamed from D?; value D52_1045 -> D
- D53: renamed from D?; value D53 -> D
- D54: renamed from D?; value D54 -> D
- D55: renamed from D?; value D55 -> D
- D56: renamed from D?; value D56 -> D
- D57: renamed from D?; value D57 -> D
- D58: renamed from D?; value D58 -> D
- D59: renamed from D?; value D59 -> D
- D6: renamed from D?; value D6 -> D
- D60: renamed from D?; value D60 -> D
- D61: renamed from D?; value D61 -> D
- D62: renamed from D?; value D62 -> D
- D62_105: renamed from D?; value D62_105 -> D
- D7: renamed from D?; value D7 -> D
- D8: renamed from D?; value D8 -> D
- D9: renamed from D?; value D9 -> D
- SD1: renamed from D?; value SD1 -> D
- SD2: renamed from D?; value SD2 -> D
- SD3: renamed from D?; value SD3 -> D
- SD4: renamed from D?; value SD4 -> D
- gave numbers to parts that had none: 6
Connections:
- wire segments 582 -> 695
Other:
- note added: "SPI1_MISO"
- note added: "SPI1_MOSI"
- note added: "SPI1_SCK"
- note added: "SPI1_SEL"
- moved on the sheet: U1

Commit message: Add pok3r LED matrix, mostly done
Parts:
- added C10, C11, C13, C27, C28, C7: C, symbol C
- added C23, C24: 10u, symbol C
- added D? (x70): LED, symbol LED
- added LR1, LR10, LR11, LR12, LR13, LR14, LR15, LR16, LR17, LR18, LR19, LR2, LR20, LR21, LR22, LR23, LR24, LR25, LR26, LR27, LR28, LR29, LR3, LR30, LR31, LR32, LR33, LR34, LR35, LR36, LR37, LR38, LR39, LR4, LR40, LR41, LR42, LR43, LR44, LR45, LR46, LR47, LR48, LR49, LR5, LR50, LR51, LR52, LR53, LR54, LR55, LR56, LR57, LR58, LR59, LR6, LR60, LR61, LR62, LR63, LR64, LR65, LR66, LR7, LR8, LR9: 15k, symbol R
- added Q1, Q10, Q11, Q12, Q13, Q14, Q15, Q16, Q17, Q2, Q3, Q4, Q5, Q6, Q7, Q8, Q9: NPN, symbol NPN
- added Q18, Q19, Q20, Q21, Q22, Q23, Q24, Q25, Q26, Q27, Q28, Q29, Q30, Q31, Q32, Q33, Q34: PNP, symbol PNP
- added Q36: Q_SOT23, symbol Q_SOT23
- added R112: 18k, symbol R
- added R113, R118: 5.1k, symbol R
- added R117: 9.1k, symbol R
- added R90, R? (x16): 2.7k, symbol R
- added R91, R? (x16): 820, symbol R
- added R92, R? (x16): 10, symbol R
- added R93, R? (x16): 4.7k, symbol R
- added U4: 74LV164, symbol 74LV164
- added U?: MCP1700-3302E_SOT23, TO_SOT_Packages_SMD:SOT-23, symbol MCP1700-3302E_SOT23
- added U? (x2): APL5932A, symbol APL5932A
Connections:
- net labels added: 2.2V, 3.5V, LCOL1, LCOL2, LCOL3, LCOL4, LCOL5, LCOL6, LCOL7, LCOL8, LROW1, LROW2, LROW3, LROW4, LROW5, LROW6, LROW7, LROW8, LROW9, TCOL1, TCOL2, TCOL3, TCOL4, TCOL5, TCOL6, TCOL7, TCOL8, TROW1, TROW2, TROW3, TROW4, TROW5, TROW6, TROW7, TROW8, TROW9
- wire segments 695 -> 1866
- no-connect marks 0 -> 1
Other:
- note added: "+"
- note added: "CAPS"
- moved on the sheet: CN1, D1, D10, D11, D12, D13, D14, D15, D16, D17, D18, D19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

Commit message: upgrade to kicad 5
Parts:
- C10, C11, C13, C23, C24, C27, C28, C7: symbol C -> chaos-device:C
- CN1: symbol USB_OTG -> pok3r-rescue:USB_OTG
- CN2: symbol CONN_01X05 -> pok3r-rescue:CONN_01X05
- D1, D10, D11, D12, D13, D14, D15, D16, D17, D18, D19, D2, D20, D21, D22, D23, D24, D25_1045, D26, D27, D28, D29, D3, D30, D31, D32, D33, D34, D35, D36, D37, D38, D39, D4, D40, D41, D42, D43, D44, D45, D46_1045, D47, D48, D49, D5, D50, D51, D52_1045, D53, D54, D55, D56, D57, D58, D59, D6, D60, D61, D62, D62_105, D7, D8, D9, SD1, SD2, SD3, SD4: symbol D -> chaos-device:D
- D? (x70): symbol LED -> chaos-device:LED
- K1, K10, K11, K12, K13, K14, K15, K16, K17, K18, K19, K2, K20, K21, K22, K23, K24, K25_104, K25_105, K26, K27, K28, K29, K3, K30, K31, K32, K33, K34, K35, K36, K37, K38, K39, K4, K40, K41, K42, K43, K44, K45, K46_104, K46_105, K47, K48, K49, K5, K50, K51, K52_104, K52_105, K53, K54, K55, K56, K57, K58, K59, K6, K60, K61, K62, K63, K63_105, K7, K8, K9: symbol MX1A -> mx1a:MX1A
- LR1, LR10, LR11, LR12, LR13, LR14, LR15, LR16, LR17, LR18, LR19, LR2, LR20, LR21, LR22, LR23, LR24, LR25, LR26, LR27, LR28, LR29, LR3, LR30, LR31, LR32, LR33, LR34, LR35, LR36, LR37, LR38, LR39, LR4, LR40, LR41, LR42, LR43, LR44, LR45, LR46, LR47, LR48, LR49, LR5, LR50, LR51, LR52, LR53, LR54, LR55, LR56, LR57, LR58, LR59, LR6, LR60, LR61, LR62, LR63, LR64, LR65, LR66, LR7, LR8, LR9, R112, R113, R117, R118, R90, R91, R92, R93, R? (x64): symbol R -> chaos-device:R
- Q1, Q10, Q11, Q12, Q13, Q14, Q15, Q16, Q17, Q2, Q3, Q4, Q5, Q6, Q7, Q8, Q9: symbol NPN -> chaos-device:NPN
- Q18, Q19, Q20, Q21, Q22, Q23, Q24, Q25, Q26, Q27, Q28, Q29, Q30, Q31, Q32, Q33, Q34: symbol PNP -> chaos-device:PNP
- Q36: symbol Q_SOT23 -> chaos-ic:Q_SOT23
- SEL1, SEL2: symbol CONN_01X02 -> pok3r-rescue:CONN_01X02
- SW1: symbol DIP_SW_QUAD -> chaos-device:DIP_SW_QUAD
- U1: symbol GD25Q -> chaos-ic:GD25Q
- U3: symbol HT32F1655 -> chaos-ic:HT32F1655
- U4: symbol 74LV164 -> chaos-ic:74LV164
- U?: symbol MCP1700-3302E_SOT23 -> pok3r-rescue:MCP1700-3302E_SOT23
- U? (x2): symbol APL5932A -> chaos-ic:APL5932A
- Y1: symbol Crystal_GND24 -> pok3r-rescue:Crystal_GND24

Commit message: schematic library cleanup
Parts:
- CN1: symbol pok3r-rescue:USB_OTG -> Connector_Specialized:USB_OTG
- CN2: symbol pok3r-rescue:CONN_01X05 -> Connector_Generic:Conn_01x05
- SEL1, SEL2: symbol pok3r-rescue:CONN_01X02 -> Connector_Generic:Conn_01x02
- SW1: symbol chaos-device:DIP_SW_QUAD -> Switch:SW_DIP_x04
- U?: symbol pok3r-rescue:MCP1700-3302E_SOT23 -> Regulator_Linear:MCP1700-3302E_SOT23
- Y1: symbol pok3r-rescue:Crystal_GND24 -> Device:Crystal_GND24
Connections:
- wire segments 1866 -> 1865
Changed lines of the file:
@@
 encoding utf-8
 Sheet 1 1
-Title ""
+Title "Vortex Pok3r"
 Date ""
 Rev ""
@@
 $EndComp
 $Comp
-L pok3r-rescue:Crystal_GND24 Y1
+L Device:Crystal_GND24 Y1
 U 1 1 59885188
 P 26400 21900
@@
 $EndComp
 $Comp
-L pok3r-rescue:3.3V #PWR04
+L power:+3.3V #PWR04
 U 1 1 5988C374
 P 24950 16850
@@
 $EndComp
 $Comp
-L pok3r-rescue:3.3V #PWR05
+L power:+3.3V #PWR05
 U 1 1 5988E038
 P 31500 17100
@@
 $EndComp
 $Comp
-L chaos-device:DIP_SW_QUAD SW1
+L Switch:SW_DIP_x04 SW1
 U 1 1 5989CF04
-P 17950 5200
-F 0 "SW1" H 18250 5200 60  0000 C CNN
-F 1 "DIP_SW_QUAD" H 17950 5300 60  0001 C CNN
-F 2 "" H 17950 5200 60  0001 C CNN
-F 3 "" H 17950 5200 60  0001 C CNN
-	1    17950 5200
-	1    0    0    -1
+P 18000 4900
+F 0 "SW1" H 18000 5250 60  0000 C CNN
+F 1 "DIP_SW_QUAD" H 18000 5000 60  0001 C CNN
+F 2 "" H 18000 4900 60  0001 C CNN
+F 3 "" H 18000 4900 60  0001 C CNN
+	1    18000 4900
+	0    -1   -1   0
 $EndComp
 $Comp
@@
 UR0_RX
 $Comp
-L pok3r-rescue:CONN_01X02 SEL2
+L Connector_Generic:Conn_01x02 SEL2
 U 1 1 598B8416
-P 28950 19450
-F 0 "SEL2" H 28950 19600 50  0000 C CNN
-F 1 "CONN_01X02" V 29050 19450 50  0001 C CNN
-F 2 "" H 28950 19450 50  0001 C CNN
-F 3 "" H 28950 19450 50  0001 C CNN
-	1    28950 19450
+P 28950 19400
+F 0 "SEL2" H 28950 19500 50  0000 C CNN
+F 1 "CONN_01X02" V 29050 19400 50  0001 C CNN
+F 2 "" H 28950 19400 50  0001 C CNN
+F 3 "" H 28950 19400 50  0001 C CNN
+	1    28950 19400
 	1    0    0    -1
 $EndComp
 $Comp
-L pok3r-rescue:CONN_01X02 SEL1
+L Connector_Generic:Conn_01x02 SEL1
 U 1 1 598B8797
-P 28950 19800
-F 0 "SEL1" H 28950 19950 50  0000 C CNN
-F 1 "CONN_01X02" V 29050 19800 50  0001 C CNN
-F 2 "" H 28950 19800 50  0001 C CNN
-F 3 "" H 28950 19800 50  0001 C CNN
-	1    28950 19800
+P 28950 19750
+F 0 "SEL1" H 28950 19850 50  0000 C CNN
+F 1 "CONN_01X02" V 29050 19750 50  0001 C CNN
+F 2 "" H 28950 19750 50  0001 C CNN
+F 3 "" H 28950 19750 50  0001 C CNN
+	1    28950 19750
 	1    0    0    -1
 $EndComp
@@
 Text GLabel 26200 16100 1    60   Input ~ 0
 ROW9
-Text GLabel 17400 5900 0    60   Input ~ 0
+Text GLabel 17400 5300 0    60   Input ~ 0
 ROW9
 $Comp
-L pok3r-rescue:CONN_01X05 CN2
+L Connector_Generic:Conn_01x05 CN2
 U 1 1 599639EC
 P 28950 18900
@@
 $EndComp
 $Comp
-L pok3r-rescue:USB_OTG CN1
+L Connector_Specialized:USB_OTG CN1
 U 1 1 59964436
 P 19800 19400
@@
 $EndComp
 $Comp
-L pok3r-rescue:3.3V #PWR08
+L power:+3.3V #PWR08
 U 1 1 59969041
 P 28650 18600
@@
 Text Notes 29100 19000 1    60   ~ 0
 Debug
-Text Notes 18500 5500 1    60   ~ 0
+Text Notes 18350 5250 1    60   ~ 0
 DIP Switches
 Text Notes 25600 17050 1    40   ~ 0
@@
 $EndComp
 $Comp
-L pok3r-rescue:MCP1700-3302E_SOT23 U?
+L Regulator_Linear:MCP1700-3302E_SOT23 U?
 U 1 1 5AE43990
 P 21200 18600
@@
 $EndComp
 $Comp
-L pok3r-rescue:3.3V #PWR?
+L power:+3.3V #PWR?
 U 1 1 5AE49AB2
 P 21800 18500
@@
 	31500 17250 31500 17100
 Wire Wire Line
-	17800 5800 17800 5900
+	17800 5200 17800 5300
 Wire Wire Line
-	17400 5900 17800 5900
+	17400 5300 17800 5300
 Wire Wire Line
-	17800 5900 17900 5900
+	17800 5300 17900 5300
 Wire Wire Line
-	17900 5900 18000 5900
+	17900 5300 18000 5300
 Wire Wire Line
-	18000 5900 18100 5900
+	18000 5300 18100 5300
 Wire Wire Line
-	18100 5900 18100 5800
+	18100 5300 18100 5200
 Wire Wire Line
-	18000 5800 18000 5900
-Connection ~ 18000 5900
+	18000 5200 18000 5300
+Connection ~ 18000 5300
 Wire Wire Line
-	17900 5900 17900 5800
-Connection ~ 17900 5900
-Connection ~ 17800 5900
+	17900 5300 17900 5200
+Connection ~ 17900 5300
+Connection ~ 17800 5300
 Wire Wire Line
 	18000 4600 18000 4350
@@
 	23700 19500 20100 19500
 Wire Wire Line
-	19700 19800 19800 19800
-Wire Wire Line
 	19800 19800 19800 19950
-Connection ~ 19800 19800
 Wire Wire Line
 	27400 18800 28750 18800
