File: vortex-tester.sch (KiCad schematic (older format))
At the start: 96 parts

Commit message: schematic library cleanup
Parts:
- D? (x47): symbol LED_RAGB -> chaos-device:LED_RAGB
- D? (x22): symbol D -> chaos-device:D
- S? (x22): symbol MX1A -> mx1a:MX1A
- U?: symbol HT32F1654 -> chaos-ic:HT32F1654
- U? (x2): symbol MBIA043GP -> chaos-ic:MBIA043GP
- U?: symbol GD25Q -> chaos-ic:GD25Q
- U?: symbol HCT138 -> chaos-ic:HCT138
Connections:
- wire segments 186 -> 187

Commit message: pok3r_rgb: RGB matrix and LED drivers
Parts:
- removed U?: HCT138, MODULE, symbol chaos-ic:HCT138
- added CN4, CN5: USB_OTG, symbol Connector_Specialized:USB_OTG
- added R104, R105, R106, R107, R108, R109: 10k, symbol chaos-device:R
- added R314, R315, R316: R, symbol chaos-device:R
- added R59, R60: 27, symbol chaos-device:R
- gave numbers to parts that had none: 1
Connections:
- net labels added: +3.3V, +5V, SPI1_MISO, SPI1_MOSI, SPI1_SCK, SPI1_SEL, USR0_RX, USR0_TX
- net labels removed: COL3, COL5
- wire segments 187 -> 227
Other:
- moved on the sheet: U6, U?
