File: pok3r-rgb2.sch (KiCad schematic (older format))
At the start: 194 parts, among them CN3 Conn_01x05, CN5 USB_OTG, K46_? MX1A, SW1 DIP_SW_QUAD, U10 MCP1700-3302E_SOT23, U3 HT32F1654, U5 GD25Q, U7 MBIA043GP, U8 MBIA043GP

Commit message: Update footprints
Parts:
- CN3: footprint (none) -> Connector_PinHeader_2.54mm:PinHeader_1x05_P2.54mm_Vertical
- CN5: footprint (none) -> Connector_USB:USB_Mini-B_Wuerth_65100516121_Horizontal
- D211, D212, D213: footprint (none) -> Diode_SMD:D_SMA
- U3: footprint MODULE -> Package_QFP:LQFP-64_7x7mm_P0.4mm
- U5: footprint MODULE -> Package_SO:SOIC-8_3.9x4.9mm_P1.27mm
- U7, U8: footprint MODULE -> Package_SO:SSOP-24_3.9x8.7mm_P0.635mm
- gave numbers to parts that had none: 118
