File: pok3r_rgb2/pok3r-rgb2.sch (KiCad schematic (older format))
At the start: 194 parts, among them CN3 Conn_01x05, CN5 USB_OTG, K1 MX1A, K10 MX1A, K11 MX1A, K12 MX1A, K13 MX1A, K14 MX1A, K15 MX1A, K16 MX1A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

Commit message: Reorganize kicad files
Parts:
- D0, D1, D10, D11, D12, D13, D14, D15, D16, D17, D18, D182, D184, D186, D188, D19, D2, D20, D21, D210, D22, D23, D24, D25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: footprint (none) -> Diode_SMD:D_SMA
- SW1: footprint (none) -> Button_Switch_THT:SW_DIP_SPSTx04_Slide_6.7x11.72mm_W7.62mm_P2.54mm_LowProfile
