File: pok3r_rgb2/pok3r-rgb2.kicad_sch (KiCad schematic)
At the start: 297 parts, among them CN1 USB_OTG, CN3 Conn_01x05, K1 MX1A, K10 MX1A, K11 MX1A, K12 MX1A, K13 MX1A, K14 MX1A, K15 MX1A, K16 MX1A, K17 MX1A, K18 MX1A, K19 MX1A, K2 MX1A, K20 MX1A, K21 MX1A, K22 MX1A, K23 MX1A, K24 MX1A, K25 MX1A, K26 MX1A, K27 MX1A, K28 MX1A, K29 MX1A, K3 MX1A, K30 MX1A, K31 MX1A, K32 MX1A, K33 MX1A, K34 MX1A, K35 MX1A, K36 MX1A, K37 MX1A, K38 MX1A, K39 MX1A, K4 MX1A, K40 MX1A, K41 MX1A, K42 MX1A, K43 MX1A, K44 MX1A, K45 MX1A, K46 MX1A, K46_1 MX1A, K46_2 MX1A, K47 MX1A, K48 MX1A, K49 MX1A, K5 MX1A, K50 MX1A, K51 MX1A, K52 MX1A, K53 MX1A, K54 MX1A, K55 MX1A, K56 MX1A, K57 MX1A, K58 MX1A, K59 MX1A, K6 MX1A, K60 MX1A, K61 MX1A, K62 MX1A, K63 MX1A, K64 MX1A, K65 MX1A, K7 MX1A, K8 MX1A, K9 MX1A, Q1 Q_NPN_BCE, Q2 Q_NPN_BCE, Q3 Q_NPN_BCE, Q4 Q_NPN_BCE, Q5 Q_NPN_BCE, Q6 Q_NPN_BCE, Q7 Q_NPN_BCE, Q73 Q_NPN_BCE, Q8 Q_NPN_BCE, SW1 DIP_SW_QUAD, U2 MCP1700-3302E_SOT23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

Commit message: Finish POK3R RGB 2
Parts:
- added C1, C14, C15, C16, C17, C18, C2, C3, C4: C, symbol chaos-device:C
- added R107: 0, symbol chaos-device:R
- added R29: 100k, symbol Device:R_US
- added R4, R5: ~, symbol Device:R_US
- added X1: Crystal_GND23, symbol Device:Crystal_GND23
- D412, D51, K2, K46_1, K5, K57, K6, K64: now not fitted
Connections:
- net 3.3V: now also R29.2
- net COL8: now also D20.2 (A), D413.2 (A), D69.2 (A)
- net GND: now also U3.19 (VSS33_2), U3.43 (VSS33_3), U3.56 (VSS33_4), C1.2, C14.2, C15.2, C16.2, C17.2, C18.2, C2.2, C3.2, C4.1, R4.1, R5.1, X1.2, X1.3
- net ROW4: now also R107.1; no longer K3.2
- net ROW6: now also K46_1.2, K46_2.2
- net ROW8: now also K6.2, K7.2
- net at U3.17 (CLDIO): now also C16.1
- net at U3.18 (VDD33_2): now also C17.1
- net at CN3.4 (Pin_4), U3.20 (nRST): now also C18.1, R29.1
- net at U3.21 (VBAT): now also C2.1
- net at U3.26 (XTALIN/PB14): now also C14.1, X1.1
- net at U3.27 (XTALOUT/PB15): now also C15.1, X1.4
- net at U3.28 (PD1): now also R5.2
- net at U3.29 (PD2): now also R4.2
- net at U3.42 (VDD33_3): now also C3.1
- net at U3.55 (VDD33_4): now also C4.2
- net SPI1_SCK: now reaches U3.58 (PB7), U5.6 (SCLK)
- net SPI1_MOSI: now reaches U3.59 (PB8), U5.5 (SI)
- net SPI1_MISO: now reaches U3.60 (PB9), U5.2 (SO)
- net SPI1_SEL: now reaches U3.61 (PB10), U5.1 (CS#)
- net at U3.9 (VDD33_1): now also C1.1
- new net: K3.2, R107.2
- no-connect marks 5 -> 8
Other:
- moved on the sheet: D20, D413, D50, D510, D511, D512, D52, D53, D54, D55, D56, D57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
