File: vortex_core/vortex-core.sch (KiCad schematic (older format))
At the start: 171 parts, among them CN2 Conn_01x05, CN3 USB_OTG, J3 Conn_01x07, J4 Conn_01x07, Q77 DNP PNP, U10 HT32F1654, U2 MCP1700-3302E_SOT23, U4 HCT138, U5 GD25Q, U7 MBIA043GP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

Commit message: Reorganize kicad files
Parts:
- CN3: symbol Connector_Specialized:USB_OTG -> vortex-core-rescue:USB_OTG-Connector_Specialized
Changed lines of the file:
@@
 EESchema Schematic File Version 4
-EELAYER 26 0
+EELAYER 30 0
 EELAYER END
 $Descr A1 33110 23386
@@
 $EndComp
 $Comp
-L Connector_Specialized:USB_OTG CN3
+L vortex-core-rescue:USB_OTG-Connector_Specialized CN3
 U 1 1 5A81EF6F
 P 14450 18900
