File: pok3r_rgb/pok3r-rgb.kicad_sch (KiCad schematic)
At the start: 291 parts, among them CN3 Conn_01x05, CN5 USB_OTG, J1 Conn_01x19_Female, J1 Conn_01x19_Male, K1 MX1A, K10 MX1A, K11 MX1A, K12 MX1A, K13 MX1A, K14 MX1A, K15 MX1A, K16 MX1A, K17 MX1A, K18 MX1A, K19 MX1A, K2 MX1A, K20 MX1A, K21 MX1A, K22 MX1A, K23 MX1A, K24 MX1A, K25_104 MX1A, K25_105 MX1A, K26 MX1A, K27 MX1A, K28 MX1A, K29 MX1A, K3 MX1A, K30 MX1A, K31 MX1A, K32 MX1A, K33 MX1A, K34 MX1A, K35 MX1A, K36 MX1A, K37 MX1A, K38 MX1A, K39 MX1A, K4 MX1A, K40 MX1A, K41 MX1A, K42 MX1A, K43 MX1A, K44 MX1A, K45 MX1A, K46_104 MX1A, K46_105 MX1A, K47 MX1A, K48 MX1A, K49 MX1A, K5 MX1A, K50 MX1A, K51 MX1A, K52_104 MX1A, K52_105 MX1A, K53 MX1A, K54 MX1A, K55 MX1A, K56 MX1A, K57 MX1A, K57_1 MX1A, K58 MX1A, K59 MX1A, K6 MX1A, K60 MX1A, K61 MX1A, K62 MX1A, K63 MX1A, K7 MX1A, K8 MX1A, K9 MX1A, Q1 Q_NPN_BCE, Q2 Q_NPN_BCE, Q3 Q_NPN_BCE, Q4 Q_NPN_BCE, Q5 Q_NPN_BCE, Q6 Q_NPN_BCE, Q7 Q_NPN_BCE, Q74 Q_NPN_BCE, Q8 Q_NPN_BCE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

Commit message: Finish POK3R RGB 2
Connections:
- net DCLK: now reaches R41.1, R68.1, U11.3 (DCLK), U4.40 (PA14), U8.3 (DCLK)
- net LE: now reaches R42.1, R70.1, U11.4 (LE), U4.41 (PA15), U8.4 (LE)
Changed lines of the file:
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@@
+		)
+	)
+	(label "LE"
+		(at 668.02 463.55 0)
+		(effects
+			(font
+				(size 1.27 1.27)
+			)
+			(justify left bottom)
+		)
+	)
+	(label "DCLK"
+		(at 668.02 466.09 0)
+		(effects
+			(font
+				(size 1.27 1.27)
+			)
+			(justify left bottom)
 		)
 	)
